File: pcb.kicad_pcb (KiCad board)
At the start: 2 copper layers, 33 x 48 mm, 21 parts, among them J1 USB4110-GF-A, J2 5749181-1, J3 AVR-ISP-6, SW1 SW_DPST_x2, U1 ATmega32U2-A, Y1 Crystal_GND24

Commit message: Fix pcb dcm errors
Parts:
- J2: footprint Library:57491811 -> footprints:5749181-1
- moved J2 3.14 mm to (82.5, 109.0), turned to 180 degrees
Connections:
- J3 pad 5: Net-(J3-~{RST}) -> Net-(J1-VBUS3)
- R1 pad 1: Net-(J3-~{RST}) -> Net-(U1-PC1/~{RESET})
- SW1 pad 2: Net-(J3-~{RST}) -> Net-(J1-VBUS3)
- U1 pad 24: Net-(J1-VBUS3) -> Net-(U1-PC1/~{RESET})
Routing:
- net Net-(U1-PC1/~{RESET}): track 0.00 -> 49.1 mm
- net Net-(J1-VBUS3): track 66.6 -> 104.0 mm, vias 2 -> 4
- net Net-(J3-~{RST}): track 32.0 -> 0.00 mm, vias 2 -> 0
- net GND: track 86.4 -> 88.6 mm
