File: pcb.kicad_sch (KiCad schematic)
At the start: 21 parts, among them J1 USB4110-GF-A, J2 5749181-1, J3 AVR-ISP-6, SW1 SW_DPST_x2, U1 ATmega32U2-A, Y1 Crystal_GND24

Commit message: Fix pcb dcm errors
Parts:
- J2: footprint Library:57491811 -> footprints:5749181-1
